Commit message: Changed kr6r700sixx xacro joint locations to match kuka documentation

File: kuka_kr6_support/urdf/kr6r700sixx_macro.xacro (robot description, xacro)
@@ -49,5 +49,5 @@
     <link name="${prefix}link_2">
       <visual>
-        <origin xyz="0 0 0" rpy="0 ${pi/2} 0" />
+        <origin xyz="0 0 0" rpy="0 0 0" />
         <geometry>
           <mesh filename="package://kuka_kr6_support/meshes/kr6r700sixx/visual/link_2.stl" />
@@ -56,5 +56,5 @@
       </visual>
       <collision>
-        <origin xyz="0 0 0" rpy="0 ${pi/2} 0" />
+        <origin xyz="0 0 0" rpy="0 0 0" />
         <geometry>
           <mesh filename="package://kuka_kr6_support/meshes/kr6r700sixx/collision/link_2.stl" />
@@ -126,5 +126,5 @@
     <!-- joints -->
     <joint name="${prefix}joint_a1" type="revolute">
-      <origin xyz="0.000 0.000 0.217" rpy="0 0 0"/>
+      <origin xyz="0 0 0.4" rpy="0 0 0"/>
       <parent link="${prefix}base_link"/>
       <child link="${prefix}link_1"/>
@@ -133,5 +133,5 @@
     </joint>
     <joint name="${prefix}joint_a2" type="revolute">
-      <origin xyz="0.025 0.000 0.183" rpy="0 0 0"/>
+      <origin xyz="0.025 0 0" rpy="0 0 0"/>
       <parent link="${prefix}link_1"/>
       <child link="${prefix}link_2"/>
@@ -140,5 +140,5 @@
     </joint>
     <joint name="${prefix}joint_a3" type="revolute">
-      <origin xyz="0.315 0.000 0.000" rpy="0 0 0"/>
+      <origin xyz="0.315 0 0" rpy="0 0 0"/>
       <parent link="${prefix}link_2"/>
       <child link="${prefix}link_3"/>
@@ -147,5 +147,5 @@
     </joint>
     <joint name="${prefix}joint_a4" type="revolute">
-      <origin xyz="0.107 0.000 0.035" rpy="0 0 0"/>
+      <origin xyz="0 0 0.035" rpy="0 0 0"/>
       <parent link="${prefix}link_3"/>
       <child link="${prefix}link_4"/>
@@ -154,5 +154,5 @@
     </joint>
     <joint name="${prefix}joint_a5" type="revolute">
-      <origin xyz="0.258 0.000 0.000" rpy="0 0 0"/>
+      <origin xyz="0.365 0 0" rpy="0 0 0"/>
       <parent link="${prefix}link_4"/>
       <child link="${prefix}link_5"/>
@@ -161,5 +161,5 @@
     </joint>
     <joint name="${prefix}joint_a6" type="revolute">
-      <origin xyz="0.080 0.000 0.000" rpy="0 0 0"/>
+      <origin xyz="0.080 0 0" rpy="0 0 0"/>
       <parent link="${prefix}link_5"/>
       <child link="${prefix}link_6"/>
@@ -168,5 +168,5 @@
     </joint>
     <joint name="${prefix}base_link-base" type="fixed">
-      <origin xyz="0.000 0.000 0.000" rpy="0 0 0"/>
+      <origin xyz="0 0 0" rpy="0 0 0"/>
       <parent link="${prefix}base_link"/>
       <child link="${prefix}base"/>
@@ -175,5 +175,5 @@
       <parent link="${prefix}link_6"/>
       <child link="${prefix}tool0"/>
-      <origin xyz="0.000 0.000 0.000" rpy="0 ${90*deg} 0"/>
+      <origin xyz="0 0 0" rpy="0 ${90*deg} 0"/>
     </joint>
   </xacro:macro>

Commit message: kr6_support: minor changes to R700 sixx xacro macro.
 - use material definitions from kuka_resources package
 - use shared DEG2RAD constant from kuka_resources
 - slight re-ordering of links and joints to bring the macro more
   in-line with the others in this package

File: kuka_kr6_support/urdf/kr6r700sixx_macro.xacro (robot description, xacro)
@@ -1,20 +1,7 @@
 <?xml version="1.0"?>
 <robot xmlns:xacro="http://ros.org/wiki/xacro">
-  <property name="pi" value="3.141592654"/>
-  <!--degrees to radians-->
-  <property name="deg" value="0.017453293"/>
-  <!-- borrowed from ros-industrial/kuka_experimental/kuka_resources/urdf/common_colours.xacro -->
-  <material name="color_kuka_pedestal">
-    <color rgba="${129/255} ${120/255} ${ 99/255 } 1.0"/>
-  </material>
-  <material name="color_kuka_orange">
-    <color rgba="${246/255} ${120/255} ${ 40/255 } 1.0"/>
-  </material>
-  <material name="color_kuka_black">
-    <color rgba="${ 14/255 } ${ 14/255 } ${ 16/255 } 1.0"/>
-  </material>
+  <xacro:include filename="$(find kuka_resources)/urdf/common_constants.xacro"/>
+  <xacro:include filename="$(find kuka_resources)/urdf/common_materials.xacro"/>
   <xacro:macro name="kuka_kr6r700sixx" params="prefix">
-    <!-- link list -->
-    <link name="${prefix}base" />
     <link name="${prefix}base_link">
       <visual>
@@ -23,5 +10,5 @@
           <mesh filename="package://kuka_kr6_support/meshes/kr6r700sixx/visual/base_link.stl" />
         </geometry>
-        <material name="color_kuka_pedestal" />
+        <xacro:material_kuka_pedestal />
       </visual>
       <collision>
@@ -38,5 +25,5 @@
           <mesh filename="package://kuka_kr6_support/meshes/kr6r700sixx/visual/link_1.stl" />
         </geometry>
-        <material name="color_kuka_orange" />
+        <xacro:material_kuka_orange />
       </visual>
       <collision>
@@ -53,5 +40,5 @@
           <mesh filename="package://kuka_kr6_support/meshes/kr6r700sixx/visual/link_2.stl" />
         </geometry>
-        <material name="color_kuka_orange" />
+        <xacro:material_kuka_orange />
       </visual>
       <collision>
@@ -68,5 +55,5 @@
           <mesh filename="package://kuka_kr6_support/meshes/kr6r700sixx/visual/link_3.stl" />
         </geometry>
-        <material name="color_kuka_orange" />
+        <xacro:material_kuka_orange />
       </visual>
       <collision>
@@ -83,5 +70,5 @@
           <mesh filename="package://kuka_kr6_support/meshes/kr6r700sixx/visual/link_4.stl" />
         </geometry>
-        <material name="color_kuka_orange" />
+        <xacro:material_kuka_orange />
       </visual>
       <collision>
@@ -98,5 +85,5 @@
           <mesh filename="package://kuka_kr6_support/meshes/kr6r700sixx/visual/link_5.stl" />
         </geometry>
-        <material name="color_kuka_orange" />
+        <xacro:material_kuka_orange />
       </visual>
       <collision>
@@ -113,5 +100,5 @@
           <mesh filename="package://kuka_kr6_support/meshes/kr6r700sixx/visual/link_6.stl" />
         </geometry>
-        <material name="color_kuka_pedestal" />
+        <xacro:material_kuka_pedestal />
       </visual>
       <collision>
@@ -122,7 +109,6 @@
       </collision>
     </link>
+    <!-- This frame corresponds to the $FLANGE coordinate system in KUKA KRC controllers. -->
     <link name="${prefix}tool0" />
-    <!-- end of link list -->
-    <!-- joints -->
     <joint name="${prefix}joint_a1" type="revolute">
       <origin xyz="0 0 0.4" rpy="0 0 0"/>
@@ -130,5 +116,5 @@
       <child link="${prefix}link_1"/>
       <axis xyz="0 0 -1"/>
-      <limit lower="${-170*deg}" upper="${170*deg}" effort="0" velocity="${360*deg}"/>
+      <limit lower="${-170 * DEG2RAD}" upper="${170 * DEG2RAD}" effort="0" velocity="${360 * DEG2RAD}"/>
     </joint>
     <joint name="${prefix}joint_a2" type="revolute">
@@ -137,5 +123,5 @@
       <child link="${prefix}link_2"/>
       <axis xyz="0 1 0"/>
-      <limit lower="${-190*deg}" upper="${45*deg}" effort="0" velocity="${300*deg}"/>
+      <limit lower="${-190 * DEG2RAD}" upper="${45 * DEG2RAD}" effort="0" velocity="${300 * DEG2RAD}"/>
     </joint>
     <joint name="${prefix}joint_a3" type="revolute">
@@ -144,5 +130,5 @@
       <child link="${prefix}link_3"/>
       <axis xyz="0 1 0"/>
-      <limit lower="${-120*deg}" upper="${156*deg}" effort="0" velocity="${360*deg}"/>
+      <limit lower="${-120 * DEG2RAD}" upper="${156 * DEG2RAD}" effort="0" velocity="${360 * DEG2RAD}"/>
     </joint>
     <joint name="${prefix}joint_a4" type="revolute">
@@ -151,5 +137,5 @@
       <child link="${prefix}link_4"/>
       <axis xyz="-1 0 0"/>
-      <limit lower="${-185*deg}" upper="${185*deg}" effort="0" velocity="${381*deg}"/>
+      <limit lower="${-185 * DEG2RAD}" upper="${185 * DEG2RAD}" effort="0" velocity="${381 * DEG2RAD}"/>
     </joint>
     <joint name="${prefix}joint_a5" type="revolute">
@@ -158,5 +144,5 @@
       <child link="${prefix}link_5"/>
       <axis xyz="0 1 0"/>
-      <limit lower="${-120*deg}" upper="${120*deg}" effort="0" velocity="${388*deg}"/>
+      <limit lower="${-120 * DEG2RAD}" upper="${120 * DEG2RAD}" effort="0" velocity="${388 * DEG2RAD}"/>
     </joint>
     <joint name="${prefix}joint_a6" type="revolute">
@@ -165,6 +151,13 @@
       <child link="${prefix}link_6"/>
       <axis xyz="-1 0 0"/>
-      <limit lower="${-350*deg}" upper="${350*deg}" effort="0" velocity="${615*deg}"/>
+      <limit lower="${-350 * DEG2RAD}" upper="${350 * DEG2RAD}" effort="0" velocity="${615 * DEG2RAD}"/>
     </joint>
+    <joint name="${prefix}joint_a6-tool0" type="fixed">
+      <parent link="${prefix}link_6"/>
+      <child link="${prefix}tool0"/>
+      <origin xyz="0 0 0" rpy="0 ${90 * DEG2RAD} 0"/>
+    </joint>
+    <!-- ROS base_link to KUKA $ROBROOT coordinate system transform -->
+    <link name="${prefix}base" />
     <joint name="${prefix}base_link-base" type="fixed">
       <origin xyz="0 0 0" rpy="0 0 0"/>
@@ -172,9 +165,4 @@
       <child link="${prefix}base"/>
     </joint>
-    <joint name="${prefix}link_6-tool0" type="fixed">
-      <parent link="${prefix}link_6"/>
-      <child link="${prefix}tool0"/>
-      <origin xyz="0 0 0" rpy="0 ${90*deg} 0"/>
-    </joint>
   </xacro:macro>
 </robot>
